File: half-swept.kicad_pcb (KiCad board)
At the start: 2 copper layers, 109 x 86.9 mm, 25 parts, among them J2 AudioJack4dpb, SW1 SW_Push, SW10 SW_Push, SW11 SW_Push, SW12 SW_Push, SW13 SW_Push, SW14 SW_Push, SW15 SW_Push, SW16 SW_Push, SW17 SW_Push, SW2 SW_Push, SW3 SW_Push, SW4 SW_Push, SW5 SW_Push, SW6 SW_Push, SW7 SW_Push, SW8 SW_Push, SW9 SW_Push, U1 ProMicro-kbd

Commit message: (new) added custom library for switches
Parts:
- SW1, SW10, SW11, SW12, SW13, SW14, SW15, SW16, SW17, SW2, SW3, SW4, SW5, SW6, SW7, SW8, SW9: footprint * duckyb-collection:SW_PG1350_rev_DPB -> library:SW_PG1350_rev_DPB
Connections:
- RSW2 pad 1: gnd -> reset
- RSW2 pad 2: gnd -> reset
